File: schematic/magazine/magazine/magazine.sch (KiCad schematic (older format))
At the start: 15 parts

Commit message: clean up repo add magazine schematic gnd both arduino in the schematic
Parts:
- removed C?: C, symbol Device:C
- removed Q? (x2): PN2222A, Package_TO_SOT_THT:TO-92_Inline, symbol Transistor_BJT:PN2222A
- removed R? (x4): R, symbol Device:R
- removed U?: prox_sensor, symbol custom:prox_sensor
- R?: value R -> 470
Connections:
- wire segments 77 -> 62
- no-connect marks 7 -> 21
Other:
- note removed: "to microcontroller"
