File: schematic/chamber/chamber.sch (KiCad schematic (older format))
At the start: 15 parts

Commit message: make a bunch of schematic changes
Parts:
- C?: value C -> 0.01uF
- R?: value R -> 470
- R? (x2): value R -> 100k
- R? (x2): value R -> 10k
Connections:
- net GND: now also A?.29 (GND), A?.6 (GND), A?.7 (GND)
- net VCC: now also A?.8 (VIN)
- net at R?.2: now also A?.25 (D10)
- net at A?.4 (3V3), TOF?.1 (VCC): now also U?.14 (VSS), U?.17 (VSS), U?.20 (VSS), U?.8 (VSS)
- no-connect marks 7 -> 20
Other:
- note removed: "to microcontroller"
Changed lines of the file:
@@
 P 2200 1750
 F 0 "R?" V 1993 1750 50  0000 C CNN
-F 1 "R" V 2084 1750 50  0000 C CNN
+F 1 "470" V 2084 1750 50  0000 C CNN
 F 2 "" V 2130 1750 50  0001 C CNN
 F 3 "~" H 2200 1750 50  0001 C CNN
@@
 P 5000 1750
 F 0 "R?" V 4793 1750 50  0000 C CNN
-F 1 "R" V 4884 1750 50  0000 C CNN
+F 1 "100k" V 4884 1750 50  0000 C CNN
 F 2 "" V 4930 1750 50  0001 C CNN
 F 3 "~" H 5000 1750 50  0001 C CNN
@@
 P 5650 1150
 F 0 "R?" H 5580 1104 50  0000 R CNN
-F 1 "R" H 5580 1195 50  0000 R CNN
+F 1 "10k" H 5580 1195 50  0000 R CNN
 F 2 "" V 5580 1150 50  0001 C CNN
 F 3 "~" H 5650 1150 50  0001 C CNN
@@
 P 6700 1150
 F 0 "R?" H 6630 1104 50  0000 R CNN
-F 1 "R" H 6630 1195 50  0000 R CNN
+F 1 "10k" H 6630 1195 50  0000 R CNN
 F 2 "" V 6630 1150 50  0001 C CNN
 F 3 "~" H 6700 1150 50  0001 C CNN
@@
 P 6100 1550
 F 0 "R?" H 6030 1504 50  0000 R CNN
-F 1 "R" H 6030 1595 50  0000 R CNN
+F 1 "100k" H 6030 1595 50  0000 R CNN
 F 2 "" V 6030 1550 50  0001 C CNN
 F 3 "~" H 6100 1550 50  0001 C CNN
@@
 P 7300 1800
 F 0 "C?" H 7415 1846 50  0000 L CNN
-F 1 "C" H 7415 1755 50  0000 L CNN
+F 1 "0.01uF" H 7415 1755 50  0000 L CNN
 F 2 "" H 7338 1650 50  0001 C CNN
 F 3 "~" H 7300 1800 50  0001 C CNN
@@
 Wire Wire Line
 	5150 1750 5350 1750
-Text Notes 7650 1350 0    50   ~ 0
-to microcontroller
 $Comp
 L custom:TOF_VL53L0X TOF?
@@
 	2750 4350 2500 4350
 Wire Wire Line
-	2500 4350 2500 5750
-Wire Wire Line
-	2500 5750 5250 5750
-Wire Wire Line
-	5250 5750 5250 3800
+	2500 4350 2500 5850
+Wire Wire Line
+	2500 5850 5250 5850
+Wire Wire Line
+	5250 5850 5250 3800
 Wire Wire Line
 	5250 3800 5350 3800
@@
 NoConn ~ 1850 7350
 NoConn ~ 2050 7350
-Wire Wire Line
-	850  6550 850  6650
 Connection ~ 850  6650
+Wire Wire Line
+	850  3300 3350 3300
+Wire Wire Line
+	850  3300 850  6650
+Connection ~ 3350 3300
+$Comp
+L power:VCC #PWR?
+U 1 1 5DE4C046
+P 3150 3250
+F 0 "#PWR?" H 3150 3100 50  0001 C CNN
+F 1 "VCC" H 3167 3423 50  0000 C CNN
+F 2 "" H 3150 3250 50  0001 C CNN
+F 3 "" H 3150 3250 50  0001 C CNN
+	1    3150 3250
+	1    0    0    -1
+$EndComp
+Wire Wire Line
+	3150 3250 3150 3450
+NoConn ~ 3450 3450
+NoConn ~ 3750 3850
+NoConn ~ 3750 4050
+NoConn ~ 3750 4250
+NoConn ~ 3750 4450
+NoConn ~ 3750 4550
+NoConn ~ 3750 4650
+NoConn ~ 3750 4750
+NoConn ~ 2750 3850
+NoConn ~ 2750 4050
+NoConn ~ 2750 4250
+NoConn ~ 2750 4450
+NoConn ~ 2750 4750
+Wire Wire Line
+	1850 4850 2750 4850
+Wire Wire Line
+	1850 1750 1850 4850
+Wire Wire Line
+	3150 5550 3150 5650
+Wire Wire Line
+	3150 5650 3250 5650
+Wire Wire Line
+	3250 5650 3250 5550
+Wire Wire Line
+	3350 5550 3350 5650
+Wire Wire Line
+	3350 5650 3250 5650
+Connection ~ 3250 5650
+$Comp
+L power:GND #PWR?
+U 1 1 5DDFB735
+P 3250 5700
+F 0 "#PWR?" H 3250 5450 50  0001 C CNN
+F 1 "GND" H 3400 5650 50  0000 C CNN
+F 2 "" H 3250 5700 50  0001 C CNN
+F 3 "" H 3250 5700 50  0001 C CNN
+	1    3250 5700
+	1    0    0    -1
+$EndComp
+Wire Wire Line
+	3250 5700 3250 5650
 $EndSCHEMATC

Commit message: made changes to schematic
Parts:
- added D? (x3): LED, symbol Device:LED
- added R? (x4): 1k, symbol Device:R
Connections:
- net GND: now also D?.1 (K), D?.1 (K), D?.1 (K), R?.2; no longer SW?.1
- net VCC: now also SW?.1
- net at A?.15 (D0/RX): now also R?.2
- net at A?.18 (D3), SW?.2: now also R?.1
- net at A?.21 (D6): now also R?.2
- net at A?.24 (D9): now also R?.2
- new net: D?.2 (A), R?.1 (x3)
- no-connect marks 20 -> 17
Changed lines of the file:
@@
 	4500 1650 4300 1650
 Wire Wire Line
-	1600 4150 2750 4150
-$Comp
-L power:GND #PWR?
-U 1 1 5DE16672
-P 1000 4150
-F 0 "#PWR?" H 1000 3900 50  0001 C CNN
-F 1 "GND" H 1005 3977 50  0000 C CNN
-F 2 "" H 1000 4150 50  0001 C CNN
-F 3 "" H 1000 4150 50  0001 C CNN
-	1    1000 4150
-	0    1    1    0
-$EndComp
+	1600 4150 2050 4150
 Wire Wire Line
 	1200 4150 1000 4150
@@
 NoConn ~ 3750 4650
 NoConn ~ 3750 4750
-NoConn ~ 2750 3850
 NoConn ~ 2750 4050
 NoConn ~ 2750 4250
-NoConn ~ 2750 4450
-NoConn ~ 2750 4750
 Wire Wire Line
 	1850 4850 2750 4850
@@
 Wire Wire Line
 	3250 5700 3250 5650
+$Comp
+L power:VCC #PWR?
+U 1 1 5DE87559
+P 1000 4150
+F 0 "#PWR?" H 1000 4000 50  0001 C CNN
+F 1 "VCC" H 1017 4323 50  0000 C CNN
+F 2 "" H 1000 4150 50  0001 C CNN
+F 3 "" H 1000 4150 50  0001 C CNN
+	1    1000 4150
+	1    0    0    -1
+$EndComp
+$Comp
+L Device:R R?
+U 1 1 5DE8801D
+P 2050 3900
+F 0 "R?" H 1980 3854 50  0000 R CNN
+F 1 "1k" H 1980 3945 50  0000 R CNN
+F 2 "" V 1980 3900 50  0001 C CNN
+F 3 "~" H 2050 3900 50  0001 C CNN
+	1    2050 3900
+	-1   0    0    1
+$EndComp
+Wire Wire Line
+	2050 4050 2050 4150
+Connection ~ 2050 4150
+Wire Wire Line
+	2050 4150 2750 4150
+$Comp
+L power:GND #PWR?
+U 1 1 5DE8C0B2
+P 2050 3600
+F 0 "#PWR?" H 2050 3350 50  0001 C CNN
+F 1 "GND" H 2055 3427 50  0000 C CNN
+F 2 "" H 2050 3600 50  0001 C CNN
+F 3 "" H 2050 3600 50  0001 C CNN
+	1    2050 3600
+	-1   0    0    1
+$EndComp
+Wire Wire Line
+	2050 3750 2050 3600
+$Comp
+L Device:R R?
+U 1 1 5DE90223
+P 5900 4650
+F 0 "R?" H 5830 4604 50  0000 R CNN
+F 1 "1k" H 5830 4695 50  0000 R CNN
+F 2 "" V 5830 4650 50  0001 C CNN
+F 3 "~" H 5900 4650 50  0001 C CNN
+	1    5900 4650
+	-1   0    0    1
+$EndComp
+$Comp
+L Device:R R?
+U 1 1 5DE90C69
+P 6900 4800
+F 0 "R?" H 6830 4754 50  0000 R CNN
+F 1 "1k" H 6830 4845 50  0000 R CNN
+F 2 "" V 6830 4800 50  0001 C CNN
+F 3 "~" H 6900 4800 50  0001 C CNN
+	1    6900 4800
+	-1   0    0    1
+$EndComp
+$Comp
+L Device:R R?
+U 1 1 5DE917D9
+P 6350 4700
+F 0 "R?" H 6280 4654 50  0000 R CNN
+F 1 "1k" H 6280 4745 50  0000 R CNN
+F 2 "" V 6280 4700 50  0001 C CNN
+F 3 "~" H 6350 4700 50  0001 C CNN
+	1    6350 4700
+	-1   0    0    1
+$EndComp
+$Comp
+L Device:LED D?
+U 1 1 5DE92202
+P 6350 5150
+F 0 "D?" V 6389 5033 50  0000 R CNN
+F 1 "LED" V 6298 5033 50  0000 R CNN
+F 2 "" H 6350 5150 50  0001 C CNN
+F 3 "~" H 6350 5150 50  0001 C CNN
+	1    6350 5150
+	0    -1   -1   0
+$EndComp
+$Comp
+L Device:LED D?
+U 1 1 5DE93D19
+P 6900 5200
+F 0 "D?" V 6939 5083 50  0000 R CNN
+F 1 "LED" V 6848 5083 50  0000 R CNN
+F 2 "" H 6900 5200 50  0001 C CNN
+F 3 "~" H 6900 5200 50  0001 C CNN
+	1    6900 5200
+	0    -1   -1   0
+$EndComp
+$Comp
+L Device:LED D?
+U 1 1 5DE93EEB
+P 5900 5100
+F 0 "D?" V 5939 4983 50  0000 R CNN
+F 1 "LED" V 5848 4983 50  0000 R CNN
+F 2 "" H 5900 5100 50  0001 C CNN
+F 3 "~" H 5900 5100 50  0001 C CNN
+	1    5900 5100
+	0    -1   -1   0
+$EndComp
+$Comp
+L power:GND #PWR?
+U 1 1 5DEA57A4
+P 5900 5400
+F 0 "#PWR?" H 5900 5150 50  0001 C CNN
+F 1 "GND" H 5905 5227 50  0000 C CNN
+F 2 "" H 5900 5400 50  0001 C CNN
+F 3 "" H 5900 5400 50  0001 C CNN
+	1    5900 5400
+	1    0    0    -1
+$EndComp
+$Comp
+L power:GND #PWR?
+U 1 1 5DEA654E
+P 6350 5450
+F 0 "#PWR?" H 6350 5200 50  0001 C CNN
+F 1 "GND" H 6355 5277 50  0000 C CNN
+F 2 "" H 6350 5450 50  0001 C CNN
+F 3 "" H 6350 5450 50  0001 C CNN
+	1    6350 5450
+	1    0    0    -1
+$EndComp
+$Comp
+L power:GND #PWR?
+U 1 1 5DEA6982
+P 6900 5500
+F 0 "#PWR?" H 6900 5250 50  0001 C CNN
+F 1 "GND" H 6905 5327 50  0000 C CNN
+F 2 "" H 6900 5500 50  0001 C CNN
+F 3 "" H 6900 5500 50  0001 C CNN
+	1    6900 5500
+	1    0    0    -1
+$EndComp
+Wire Wire Line
+	5900 4500 5900 4150
+Wire Wire Line
+	5900 4150 6750 4150
+Wire Wire Line
+	6750 4150 6750 3000
+Wire Wire Line
+	6750 3000 2400 3000
+Wire Wire Line
+	2400 3000 2400 3850
+Wire Wire Line
+	2400 3850 2750 3850
+Wire Wire Line
+	5900 4800 5900 4950
+Wire Wire Line
+	5900 5250 5900 5400
+Wire Wire Line
+	6350 5300 6350 5450
+Wire Wire Line
+	6900 5350 6900 5500
+Wire Wire Line
+	6900 4950 6900 5050
+Wire Wire Line
+	6350 4850 6350 5000
+Wire Wire Line
+	6350 4550 6350 4250
+Wire Wire Line
+	6350 4250 6850 4250
+Wire Wire Line
+	6850 4250 6850 2900
+Wire Wire Line
+	6850 2900 2300 2900
+Wire Wire Line
+	2300 2900 2300 4450
+Wire Wire Line
+	2300 4450 2750 4450
+Wire Wire Line
+	2750 4750 2350 4750
+Wire Wire Line
+	2350 4750 2350 5950
+Wire Wire Line
+	2350 5950 7350 5950
+Wire Wire Line
+	7350 5950 7350 4500
+Wire Wire Line
+	7350 4500 6900 4500
+Wire Wire Line
+	6900 4500 6900 4650
 $EndSCHEMATC
